Commit message: 1.remove an error from urdf files 2.make the configration of movebase more clear

File: urdf_gazebo_02/urdf/xacro/blitzcrank.urdf.xacro (robot description, xacro)
@@ -95,5 +95,5 @@
                 </geometry>
                 <origin xyz="0 0 0" rpy="${PI/2} 0 0" />
-                <material name="red" />
+                <material name="wheel_color" />
             </visual>
             <collision>

File: urdf_gazebo_02/urdf/xacro/demo05_car_base.urdf.xacro (robot description, xacro)
@@ -89,5 +89,5 @@
                 </geometry>
                 <origin xyz="0 0 0" rpy="0 0 0" />
-                <material name="red" />
+                <material name="wheel_color" />
             </visual>
             <collision>

File: urdf_gazebo_02/urdf/xacro/demo06_car_camera.urdf.xacro (robot description, xacro)
@@ -14,5 +14,5 @@
             </geometry>
             <origin xyz="0 0 0" rpy="0 0 0"/>
-            <material name="red">
+            <material name="wheel_color">
                 <color rgba="0 0 0 0.5"/>
             </material>

File: urdf_gazebo_02/urdf/xacro/demo07_car_laser.urdf.xacro (robot description, xacro)
@@ -41,5 +41,5 @@
                 <cylinder radius="${laser_radius}" length="${laser_length}"/>
             </geometry>
-            <material name="red">
+            <material name="wheel_color">
                 <color rgba="0.0 0.0 0.0 0.5"/>
             </material>

File: urdf_rviz_01/urdf/xacro/demo06_car_camera.urdf.xacro (robot description, xacro)
@@ -13,5 +13,5 @@
             </geometry>
             <origin xyz="0 0 0" rpy="0 0 0"/>
-            <material name="red">
+            <material name="wheel_color">
                 <color rgba="0 0 0 0.5"/>
             </material>

File: urdf_rviz_01/urdf/xacro/demo07_car_laser.urdf.xacro (robot description, xacro)
@@ -30,5 +30,5 @@
                 <cylinder radius="${laser_radius}" length="${laser_length}"/>
             </geometry>
-            <material name="red">
+            <material name="wheel_color">
                 <color rgba="0.0 0.0 0.0 0.5"/>
             </material>
